Commit message: Add tactile stub and MuJoCo hand backend (slices 6-7 stage 1)
Slice 6 (eFlesh tactile interface stub):
- surgical_hand_msgs/TactileState: eFlesh-shaped message (raw
  magnetometer array + contact/normal/shear/slip/location), with
  simulated and processed_valid flags as first-class fields.
- surgical_hand_tactile: ROS-free TactileSource interface +
  SimulatedTactileSource (deterministic-when-noiseless synthetic
  contact episodes; 9 gtests) + tactile_publisher node with per-
  fingertip topics. Real eFlesh later implements the same interface
  without changing topics/messages/consumers.

Slice 7 stage 1 (hand-only MuJoCo backend):
- GenericMjJointPositionHardwareSystem: optional per-joint
  mj_joint_name parameter (default = joint name; Wuji unchanged) so
  ros2_control joints can map onto differently-named MJCF joints.
- hand_joints.yaml: mj_joint field mapping ORCA URDF CAD names onto
  the MJCF semantic names; emitted by the ros2_control xacro.
- surgical_hand_mujoco.launch.py + surgical_hand_mujoco.yaml: runs
  upstream's ORCA v2 scene in mujoco_ros with the same controllers
  and topics as the mock backend. Verified headless end-to-end:
  close/precision_pinch/open track through physics.
- mujoco_ros main.cpp fix (upstreamable): headless+GLFW builds never
  spun the ROS executor, hanging every service including
  controller_manager. Spin in a background thread when headless.
- hand_pose_cli: repeat the command for 1 s instead of publishing
  once (one-shot messages were lost against the busy sim executor).

Co-Authored-By: Claude Fable 5 <noreply@anthropic.com>

File: src/surgical_hand/surgical_hand_description/robots/surgical_hand.ros2_control.xacro (robot description, xacro)
@@ -36,6 +36,11 @@
         <xacro:if value="${entries != []}">
           <xacro:property name="entry" value="${entries[0]}"/>
+          <!-- mj_joint maps to the MJCF joint name when it differs from the
+               URDF name (ORCA MJCF uses semantic names); ignored by the
+               mock backend. -->
+          <xacro:property name="mj_joint" value="${entry['mj_joint'] if 'mj_joint' in entry else entry['name']}"/>
           <joint name="${entry['name']}">
-            <param name="actuator_name">${entry['name']}_actuator</param>
+            <param name="mj_joint_name">${mj_joint}</param>
+            <param name="actuator_name">${mj_joint}_actuator</param>
             <param name="initial_position">${entry['initial_position']}</param>
             <command_interface name="position">
